Commit message: Split the camera doc into basics and one-box, drawn from Gazebo captures
The camera area is now two docs, and every picture in them is a real capture
from the camera_one_box simulation in Gazebo:

- docs/camera/basics.md: what a camera is for, pixels, what a picture loses,
  depth, the cameras used, the lens as four numbers, and field of view against
  resolution. These were sections 1.1 to 1.7.
- docs/camera/one-box.md: the problem, the calculations, pseudo code, and
  Python that uses the project's own libraries (rosbag2, cv_bridge,
  image_geometry, tf2, measure.py) on the recorded capture. Then new sections
  on how the project runs (the pieces, the two camera frames, the topics and
  the settings), running it, the code layout, gotchas and vocabulary.

The three-box example is removed, to keep the area to the basics. Images now
live in one folder per doc: docs/images/camera/basics/ and one-box/.

docs/diagrams/record_camera.py runs the simulation with six camera settings and
saves one compressed capture of each into docs/diagrams/captures/camera/.
docs/diagrams/camera.py draws from those captures, reads the box from the world
file, and turns pixels into points with measure.py. Every count and depth in
the docs matched Gazebo unchanged. Only the colours moved, because Gazebo lights
the scene: the sample pixel is (202, 121, 112), grey 144. All eight Python blocks
in one-box.md run and print what the doc says.

The camera description takes width, height and hfov_deg arguments, and so does
the launch file. The stand height argument is now mount_height, and snapshots
are zstd-compressed (the test capture went from 569 KB to 32 KB).

Removed: the old camera_basics package (ray caster, walkthroughs, publisher
node) and its tests, docs/camera/overview.md, and the old flat images. The
Makefile's camera commands are now camera.one_box, camera.pixels and
camera.check. The README, the arm doc and the tools doc link to the new docs.
The .flake8 list of this repo's own packages no longer includes arm_transforms,
which had broken make lint for the arm package.

Co-Authored-By: Claude Opus 5 <noreply@anthropic.com>
Claude-Session: https://claude.ai/code/session_014pENzTX8Fwof2SgoRfagAu

File: src/camera_one_box/urdf/camera.urdf.xacro (robot description, xacro)
@@ -9,6 +9,11 @@
 -->
 <robot name="camera_stand" xmlns:xacro="http://www.ros.org/wiki/xacro">
-  <!-- xacro already knows pi, so the angles below can use it directly. -->
-  <xacro:arg name="height" default="0.40"/>
+  <!-- How high the stand holds the camera, in metres. -->
+  <xacro:arg name="mount_height" default="0.40"/>
+  <!-- The camera: how many pixels across and down, and how wide it sees. The
+       defaults are the camera the doc uses. xacro already knows pi and radians(). -->
+  <xacro:arg name="width" default="320"/>
+  <xacro:arg name="height" default="240"/>
+  <xacro:arg name="hfov_deg" default="60"/>
   <link name="world"/>
   <!-- The camera body. Like every other link on a robot, its X points forward
@@ -36,5 +41,5 @@
     <!-- Pitch a quarter turn so the lens looks down at the table, then yaw a
          quarter turn so that world +Y comes out at the top of the picture. -->
-    <origin xyz="0 0 $(arg height)" rpy="0 ${pi / 2} ${pi / 2}"/>
+    <origin xyz="0 0 $(arg mount_height)" rpy="0 ${pi / 2} ${pi / 2}"/>
   </joint>
   <!-- The optical frame: X right, Y down the picture, Z out of the lens. It is
@@ -48,5 +53,6 @@
   </joint>
   <gazebo reference="camera_link">
-    <!-- The camera the doc uses: 320 x 240 pixels, 60 degrees across. -->
+    <!-- The camera the doc uses: 320 x 240 pixels, 60 degrees across, unless
+         the launch file asks for another. -->
     <sensor name="camera" type="rgbd_camera">
       <topic>camera</topic>
@@ -55,8 +61,8 @@
       <always_on>true</always_on>
       <camera>
-        <horizontal_fov>${pi / 3}</horizontal_fov>
+        <horizontal_fov>${radians($(arg hfov_deg))}</horizontal_fov>
         <image>
-          <width>320</width>
-          <height>240</height>
+          <width>$(arg width)</width>
+          <height>$(arg height)</height>
         </image>
         <clip>
