Commit message: Explain sensor_msgs and the camera's message classes; give the arm a gripper and a sensor
ROS intro: a new section 3, "Message types and the sensor_msgs package":

- what sensor_msgs is, and why shared definitions let drivers and programs
  from different people work together
- a table of its most common types, and the other standard message packages
- how a .msg file becomes a Python class in the package's msg module, and
  what a new message holds
- constants such as Range.INFRARED, and messages inside messages (the header)

Later sections are renumbered, and the camera doc's link into the intro
follows.

ROS camera: section 2 becomes "The camera's two message classes":

- 2.1 Image: every field, including is_bigendian, and the header.
- 2.2 CameraInfo: every field (k, distortion_model, d, r, p, binning, roi),
  what this example sends, a real `ros2 topic echo --flow-style` message, and
  what a calibrated camera fills in.

ROS arm: the smallest gripper and the smallest sensor.

- URDF: a palm, and two fingers on one prismatic joint "gripper". The second
  finger copies it with <mimic>, which robot_state_publisher follows.
- URDF: a range_sensor frame under the palm, pointing down.
- arm_mover also opens and closes the gripper, from 0 to 0.02 m.
- The new distance_sensor node looks up the sensor with TF and publishes a
  sensor_msgs/Range on /tip_range: 0.085 m when the arm is level, up to about
  0.39 m when it tilts up. RViz shows the beam.
- The follower in ros_camera_arm holds the gripper open, so RViz can draw it.
- The arm doc gains sections 6 (the gripper) and 7 (the distance sensor, with
  the Range class field by field), plus a new diagram. Tests cover the
  gripper's limits and the distance calculation.

Co-Authored-By: Claude Opus 5 <noreply@anthropic.com>
Claude-Session: https://claude.ai/code/session_014pENzTX8Fwof2SgoRfagAu

File: src/ros/ros_arm/urdf/arm.urdf (robot description, URDF)
Before this commit: robot pointer_arm, 4 links, 3 joints
Links:
- added link left_finger; visual box size=0.04 0.008 0.02
- added link range_sensor
- added link right_finger; visual box size=0.04 0.008 0.02
- link tip: geometry visual box size=0.02 0.07 0.03
Joints:
- added joint gripper: type prismatic, parent tip, child left_finger, origin xyz=0.02 0 0, axis 0 1 0, limit lower=0 upper=0.02 effort=1 velocity=0.1
- added joint gripper_mirror: type prismatic, parent tip, child right_finger, origin xyz=0.02 0 0, axis 0 -1 0, limit lower=0 upper=0.02 effort=1 velocity=0.1, mimic joint=gripper
- added joint range_sensor_joint: type fixed, parent tip, child range_sensor, origin xyz=0.01 0 -0.015 rpy=0 1.5708 0
